File: STM32F103/STM32F103_Devel/STM32103_Devel.kicad_pcb (KiCad board)
At the start: 4 copper layers, 69 x 50 mm, 45 parts, among them J1 Conn_02x03_Odd_Even, J2 USB_B_Micro, J3 Conn_02x10_Odd_Even, J4 Conn_01x16, J5 Conn_01x16, SW1 SW_Push, U1 STM32F103RBTx, U2 AMS1117-3.3, Y1 8MHz, Y2 Crystal

Commit message: STM32F103 Devel 0.0.2
Parts:
- added J6: Conn_02x05 Odd_Even, Connector_PinHeader_1.27mm:PinHeader_2x05_P1.27mm_Vertical, F.Cu at (164.9, 81.2)
- U1: value STM32F103RBTx -> STM32F103CBTx
- moved J4 42.3 mm to (109.0, 116.0), turned to 90 degrees
- moved J5 42.2 mm to (109.0, 74.0)
- moved H1 16.0 mm to (165.0, 74.0)
- moved D3 14.3 mm to (122.6, 77.2), turned to 0 degrees
- moved R6 14.1 mm to (122.6, 79.4), turned to 0 degrees
- moved J2 10.5 mm to (156.3, 73.9), turned to 180 degrees
- moved R8 8.77 mm to (145.3, 78.9), turned to 180 degrees
- moved H4 8.60 mm to (104.0, 116.0)
- moved R7 7.25 mm to (152.3, 78.9), turned to 180 degrees
- moved R5 6.92 mm to (118.6, 83.0), turned to 0 degrees
- moved H3 6.00 mm to (104.0, 74.0)
- moved J1 5.29 mm to (114.0, 80.0), turned to 270 degrees
- moved C6 4.95 mm to (135.6, 88.1), turned to 180 degrees
- moved C7 4.87 mm to (123.9, 84.8), turned to 270 degrees
- moved R1 4.45 mm to (118.6, 79.2), turned to 0 degrees
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Connections:
- net Net-(J2-Pad2) renamed /USB_N
- net Net-(J2-Pad3) renamed /USB_P
Routing:
- net /PB5: track 56.4 -> 28.2 mm
- net /PB4: track 52.6 -> 25.9 mm
- net /BOOT1: track 61.0 -> 35.0 mm, vias 3 -> 2
- net /PB6: track 50.5 -> 24.7 mm
- net /RST: track 71.9 -> 97.1 mm, vias 2 -> 3
- net /PB7: track 46.9 -> 22.2 mm
- net /PB8: track 43.5 -> 22.7 mm
- net /PB3: track 100.6 -> 79.8 mm, vias 2 -> 3
- net /PA12: track 69.7 -> 50.1 mm
- net /PA11: track 64.6 -> 45.9 mm, vias 1 -> 0
- net /PA10: track 47.6 -> 29.0 mm, vias 1 -> 0
- net /PB9: track 40.4 -> 22.8 mm
- net /PA7: track 36.8 -> 20.1 mm, vias 1 -> 0
- net /PA9: track 46.3 -> 29.8 mm, vias 1 -> 0
- net /PA8: track 45.0 -> 31.0 mm, vias 1 -> 0
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Other:
- board text added: "-3.3V"
- board text added: "-5V"
- board text added: "-PB5"
- board text added: "0"
- board text added: "0 - 1"
- board text added: "15"
- board text added: "B1"
- board text added: "Boot 0 Boot 1"
- board text added: "DCLK"
- board text added: "DIO"
- board text added: "L1"
- board text added: "TO"
- board text added: "U+"
- board text added: "U-"
