File: STM32F1/STM32F103/STM32F103CBT8_Devel/STM32103_Devel.kicad_pcb (KiCad board)
At the start: 4 copper layers, 69 x 50 mm, 45 parts, among them J2 USB_B_Micro, J4 Conn_01x16, J5 Conn_01x16, J6 Conn_02x05 Odd_Even, SW1 SW_Push, SW2 SW_DIP_x02, U1 STM32F103CBTx, U2 AMS1117-3.3, Y1 8MHz, Y2 32.768kHz

Commit message: Power Buttons
Parts:
- added J1: Conn_02x03_Counter_Clockwise, Connector_PinHeader_2.54mm:PinHeader_2x03_P2.54mm_Vertical, F.Cu at (153.0, 76.4)
- added J3: Conn_02x03_Counter_Clockwise, Connector_PinHeader_2.54mm:PinHeader_2x03_P2.54mm_Vertical, F.Cu at (165.4, 95.2)
- moved J6 4.40 mm to (163.8, 107.4)
- moved D4 4.00 mm to (154.0, 88.0)
Routing:
- net +5V: track 14.7 -> 35.1 mm
- net /USB/VCC_USB: track 11.6 -> 7.62 mm
- net /PA14: track 83.1 -> 86.8 mm
- net /PB3: track 73.5 -> 76.3 mm
- net /PA13: track 78.6 -> 81.4 mm
- net /STM32F103CB/RST: track 77.5 -> 79.1 mm
- net VCC: track 60.1 -> 59.3 mm
- net GND: vias 2 -> 9
Other:
- board text added: "3.3V"
- board text added: "5V GND"
- board text added: "GND"
- board text removed: "RST"
- board text removed: "SWDCLK"
- board text removed: "SWDIO"
- board text removed: "SWO"

Commit message: Changes
Parts:
- J2: footprint Connector_USB:USB_Micro-B_Wuerth_629105150521_CircularHoles -> Connector_USB:USB_Micro-B_Amphenol_10118193-0001LF_Horizontal
- SW1: footprint Button_Switch_THT:SW_PUSH_6mm -> STM32103_Devel:SW_PTS526_SM08_SMTR2_LFS
- SW2: footprint Button_Switch_SMD:SW_DIP_SPSTx02_Slide_6.7x6.64mm_W6.73mm_P2.54mm_LowProfile_JPin -> Button_Switch_SMD:SW_DIP_SPSTx02_Slide_6.7x6.64mm_W8.61mm_P2.54mm_LowProfile
- moved SW1 5.00 mm to (156.0, 116.0), turned to 0 degrees
- moved J2 2.26 mm to (167.5, 86.0)
- moved SW2 0.95 mm to (110.5, 81.0)
Routing:
- net /PB2: track 50.0 -> 52.1 mm
- net /STM32F103CB/BOOT0: track 29.6 -> 31.4 mm
- net /USB/VCC_USB: track 7.62 -> 9.11 mm
- net /USB/USB_P: track 21.4 -> 22.9 mm
- net /USB/USB_N: track 19.3 -> 20.8 mm
- net unconnected-(J2-ID-Pad4): track 4.20 -> 5.68 mm
Other:
- board text added: "B0 B1"
- board text removed: "Boot 0 Boot 1"
