File: STM32F1/STM32F103/STM32F103CBT8_Devel/STM32F103CB.kicad_sch (KiCad schematic)
At the start: 25 parts, among them SW2 SW_DIP_x02

Commit message: MPN from 030
Parts:
- C? (x5): LCSC C49678 -> C49678; Manufacturer (none) -> Kemet; mnp (none) -> C0805C104J5RAC7800
- C? (x2): Manufacturer (none) -> Kemet; mnp (none) -> C0805C200J5HAC7800
- C? (x2): LCSC C1785 -> C1785; Manufacturer (none) -> Kemet
- C? (x2): Manufacturer (none) -> Kemet; mnp (none) -> C0805C105J4REC7800
- C? (x2): Manufacturer (none) -> Kemet; mnp (none) -> C0805C103J5RAC7210
- J?: LCSC (none) -> C5632705; Manufacturer (none) -> Amphenol ICC (FCI); mnp (none) -> 20021121-00010C4LF
- L? (x2): LCSC C1046 -> C1046; Manufacturer (none) -> TDK Corporation; mnp (none) -> MLZ2012N100LT000
- R? (x3): LCSC C17414 -> C17414; Manufacturer (none) -> Bourns Inc.; mnp (none) -> CR0805-FX-1002ELF
- SW2: LCSC (none) -> C2921579; Manufacturer (none) -> CTS Electrocomponents; mnp (none) -> CT2192LPST-ND
- Y?: value Crystal -> 32.768kHz

Commit message: Mpn ids
Parts:
- C? (x2): mnp (none) -> C0805C100J5RACTU
- U?: Manufacturer (none) -> STM32F103CBT7; mnp (none) -> STM32F103CBT7
- Y?: Manufacturer (none) -> Abracon LLC; mnp (none) -> ABM3-8.000MHZ-B4Y-T
- Y?: Manufacturer (none) -> Abracon LLC; mnp (none) -> ABS07AIG-32.768KHZ-D-T
Changed lines of the file:
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@@
 			)
 		)
-		(property "Manufacturer" ""
+		(property "Manufacturer" "STM32F103CBT7"
 			(at 49.53 81.28 0)
 			(effects
@@
 			)
 		)
-		(property "mnp" ""
+		(property "mnp" "STM32F103CBT7"
 			(at 49.53 81.28 0)
 			(effects
@@
 			)
 		)
-		(property "Manufacturer" ""
+		(property "Manufacturer" "Abracon LLC"
 			(at 208.28 90.17 0)
 			(effects
@@
 			)
 		)
-		(property "mnp" ""
+		(property "mnp" "ABM3-8.000MHZ-B4Y-T"
 			(at 208.28 90.17 0)
 			(effects
@@
 			)
 		)
-		(property "Manufacturer" ""
+		(property "Manufacturer" "Abracon LLC"
 			(at 208.28 110.49 0)
 			(effects
@@
 			)
 		)
-		(property "mnp" ""
+		(property "mnp" "ABS07AIG-32.768KHZ-D-T"
 			(at 208.28 110.49 0)
 			(effects
@@
 			)
 		)
-		(property "mnp" ""
+		(property "mnp" "C0805C100J5RACTU"
 			(at 198.12 115.57 0)
 			(effects
@@
 			)
 		)
-		(property "mnp" ""
+		(property "mnp" "C0805C100J5RACTU"
 			(at 198.12 105.41 0)
 			(effects

Commit message: Mov USB
Parts:
- removed J?: Conn_02x10_Odd_Even, Connector_PinHeader_2.54mm:PinHeader_2x10_P2.54mm_Vertical, symbol Connector_Generic:Conn_02x10_Odd_Even
- J?: footprint Connector_PinHeader_1.27mm:PinHeader_2x05_P1.27mm_Vertical -> Connector_PinHeader_1.27mm:PinHeader_2x05_P1.27mm_Vertical_SMD
Connections:
- no-connect marks 7 -> 2
Other:
- moved on the sheet: J?

Commit message: MPN
Parts:
- C? (x5): mnp C0805C104J5RAC7800 -> (none); mpn (none) -> C0805C104J5RAC7800
- C? (x2): mnp C0805C200J5HAC7800 -> (none); mpn (none) -> C0805C200J5HAC7800
- C? (x2): mnp C0805C100J5RACTU -> (none); mpn (none) -> C0805C100J5RACTU
- C? (x2): mnp C0805C105J4REC7800 -> (none); mpn (none) -> C0805C105J4REC7800
- C? (x2): mnp C0805C103J5RAC7210 -> (none); mpn (none) -> C0805C103J5RAC7210
- J?: mnp 20021121-00010C4LF -> (none); mpn (none) -> 20021121-00010C4LF
- L? (x2): mnp MLZ2012N100LT000 -> (none); mpn (none) -> MLZ2012N100LT000
- R? (x3): mnp CR0805-FX-1002ELF -> (none); mpn (none) -> CR0805-FX-1002ELF
- SW2: mnp CT2192LPST-ND -> (none); mpn (none) -> CT2192LPST-ND
- U?: mnp STM32F103CBT7 -> (none); mpn (none) -> STM32F103CBT7
- Y?: mnp ABM3-8.000MHZ-B4Y-T -> (none); mpn (none) -> ABM3-8.000MHZ-B4Y-T
- Y?: mnp ABS07AIG-32.768KHZ-D-T -> (none); mpn (none) -> ABS07AIG-32.768KHZ-D-T
Changed lines of the file:
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@@
 			)
 		)
-		(property "mnp" "STM32F103CBT7"
+		(property "mpn" "STM32F103CBT7"
 			(at 49.53 81.28 0)
 			(effects
@@
 			)
 		)
-		(property "mnp" "C0805C104J5RAC7800"
+		(property "mpn" "C0805C104J5RAC7800"
 			(at 66.04 29.21 0)
 			(effects
@@
 			)
 		)
-		(property "mnp" "C0805C104J5RAC7800"
+		(property "mpn" "C0805C104J5RAC7800"
 			(at 54.61 29.21 0)
 			(effects
@@
 			)
 		)
-		(property "mnp" "C0805C104J5RAC7800"
+		(property "mpn" "C0805C104J5RAC7800"
 			(at 41.91 29.21 0)
 			(effects
@@
 			)
 		)
-		(property "mnp" "C0805C104J5RAC7800"
+		(property "mpn" "C0805C104J5RAC7800"
 			(at 30.48 29.21 0)
 			(effects
@@
 			)
 		)
-		(property "mnp" "ABM3-8.000MHZ-B4Y-T"
+		(property "mpn" "ABM3-8.000MHZ-B4Y-T"
 			(at 208.28 90.17 0)
 			(effects
@@
 			)
 		)
-		(property "mnp" "C0805C200J5HAC7800"
+		(property "mpn" "C0805C200J5HAC7800"
 			(at 198.12 95.25 0)
 			(effects
@@
 			)
 		)
-		(property "mnp" "C0805C200J5HAC7800"
+		(property "mpn" "C0805C200J5HAC7800"
 			(at 198.12 85.09 0)
 			(effects
@@
 			)
 		)
-		(property "mnp" "ABS07AIG-32.768KHZ-D-T"
+		(property "mpn" "ABS07AIG-32.768KHZ-D-T"
 			(at 208.28 110.49 0)
 			(effects
@@
 			)
 		)
-		(property "mnp" "C0805C100J5RACTU"
+		(property "mpn" "C0805C100J5RACTU"
 			(at 198.12 115.57 0)
 			(effects
@@
 			)
 		)
-		(property "mnp" "C0805C100J5RACTU"
+		(property "mpn" "C0805C100J5RACTU"
 			(at 198.12 105.41 0)
 			(effects
@@
 			)
 		)
-		(property "mnp" "20021121-00010C4LF"
-			(at 129.54 38.1 0)
-			(effects
-				(font
-					(size 1.27 1.27)
-				)
-				(hide yes)
-			)
-		)
 		(property "LCSC" "C5632705"
 			(at 129.54 38.1 0)
@@
 			)
 		)
+		(property "mpn" "20021121-00010C4LF"
+			(at 129.54 38.1 0)
+			(effects
+				(font
+					(size 1.27 1.27)
+				)
+				(hide yes)
+			)
+		)
 		(pin "1"
 		)
@@
 			)
 		)
-		(property "mnp" "CT2192LPST-ND"
-			(at 140.97 83.82 0)
-			(effects
-				(font
-					(size 1.27 1.27)
-				)
-				(hide yes)
-			)
-		)
 		(property "LCSC" "C2921579"
 			(at 140.97 83.82 0)
@@
 			)
 		)
+		(property "mpn" "CT2192LPST-ND"
+			(at 140.97 83.82 0)
+			(effects
+				(font
+					(size 1.27 1.27)
+				)
+				(hide yes)
+			)
+		)
 		(pin "1"
 		)
@@
 			)
 		)
-		(property "mnp" "C0805C104J5RAC7800"
+		(property "mpn" "C0805C104J5RAC7800"
 			(at 121.92 127 0)
 			(effects
@@
 			)
 		)
-		(property "mnp" ""
-			(at 133.35 127 0)
-			(effects
-				(font
-					(size 1.27 1.27)
-				)
-				(hide yes)
-			)
-		)
 		(pin "1"
 		)
@@
 			)
 		)
-		(property "mnp" "CR0805-FX-1002ELF"
+		(property "mpn" "CR0805-FX-1002ELF"
 			(at 128.27 90.17 0)
 			(effects
@@
 			)
 		)
-		(property "mnp" "CR0805-FX-1002ELF"
+		(property "mpn" "CR0805-FX-1002ELF"
 			(at 118.11 90.17 0)
 			(effects
@@
 			)
 		)
-		(property "mnp" "CR0805-FX-1002ELF"
+		(property "mpn" "CR0805-FX-1002ELF"
 			(at 142.24 120.65 0)
 			(effects
@@
 			)
 		)
-		(property "mnp" "C0805C105J4REC7800"
+		(property "mpn" "C0805C105J4REC7800"
 			(at 190.5 39.37 0)
 			(effects
@@
 			)
 		)
-		(property "mnp" "C0805C103J5RAC7210"
+		(property "mpn" "C0805C103J5RAC7210"
 			(at 200.66 39.37 0)
 			(effects
@@
 			)
 		)
-		(property "mnp" "C0805C105J4REC7800"
+		(property "mpn" "C0805C105J4REC7800"
 			(at 218.44 39.37 0)
 			(effects
@@
 			)
 		)
-		(property "mnp" "C0805C103J5RAC7210"
+		(property "mpn" "C0805C103J5RAC7210"
 			(at 228.6 39.37 0)
 			(effects
@@
 			)
 		)
-		(property "mnp" "MLZ2012N100LT000"
+		(property "mpn" "MLZ2012N100LT000"
 			(at 209.55 45.72 0)
 			(effects
@@
 			)
 		)
-		(property "mnp" "MLZ2012N100LT000"
+		(property "mpn" "MLZ2012N100LT000"
 			(at 209.55 34.29 0)
 			(effects

Commit message: Changes
Parts:
- SW2: footprint Button_Switch_SMD:SW_DIP_SPSTx02_Slide_6.7x6.64mm_W6.73mm_P2.54mm_LowProfile_JPin -> Button_Switch_SMD:SW_DIP_SPSTx02_Slide_6.7x6.64mm_W8.61mm_P2.54mm_LowProfile; LCSC C2921579 -> C2842684; mpn CT2192LPST-ND -> 219-2LPST
- SW?: footprint Button_Switch_THT:SW_PUSH_6mm -> STM32103_Devel:SW_PTS526_SM08_SMTR2_LFS; LCSC (none) -> C2689521; MPN (none) -> PTS526 SK15 SMTR2 LFS; Manufacturer (none) -> C&K; mpn (none) -> PTS526 SK15 SMTR2 LFS
Changed lines of the file:
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@@
 			)
 		)
-		(property "Footprint" "Button_Switch_SMD:SW_DIP_SPSTx02_Slide_6.7x6.64mm_W6.73mm_P2.54mm_LowProfile_JPin"
+		(property "Footprint" "Button_Switch_SMD:SW_DIP_SPSTx02_Slide_6.7x6.64mm_W8.61mm_P2.54mm_LowProfile"
 			(at 140.97 83.82 0)
 			(effects
@@
 			)
 		)
-		(property "LCSC" "C2921579"
-			(at 140.97 83.82 0)
-			(effects
-				(font
-					(size 1.27 1.27)
-				)
-				(hide yes)
-			)
-		)
-		(property "mpn" "CT2192LPST-ND"
+		(property "LCSC" "C2842684"
+			(at 140.97 83.82 0)
+			(effects
+				(font
+					(size 1.27 1.27)
+				)
+				(hide yes)
+			)
+		)
+		(property "mpn" "219-2LPST"
 			(at 140.97 83.82 0)
 			(effects
@@
 		)
 		(pin "4"
+		)
+		(instances
+			(project ""
+				(path "/85ec8920-663a-4b80-8ed7-b7d8c4fb3d9b/00000000-0000-0000-0000-00006115f145"
+					(reference "SW2")
+					(unit 1)
+				)
+			)
 		)
 	)
@@
 			)
 		)
-		(property "Footprint" "Button_Switch_THT:SW_PUSH_6mm"
+		(property "Footprint" "STM32103_Devel:SW_PTS526_SM08_SMTR2_LFS"
 			(at 138.43 127 0)
 			(effects
@@
 			)
 		)
-		(property "Manufacturer" ""
+		(property "Manufacturer" "C&K"
 			(at 133.35 127 0)
 			(effects
+				(font
+					(size 1.27 1.27)
+				)
+				(hide yes)
+			)
+		)
+		(property "MPN" "PTS526 SK15 SMTR2 LFS"
+			(at 133.35 127 90)
+			(effects
+				(font
+					(size 1.27 1.27)
+				)
+				(hide yes)
+			)
+		)
+		(property "mpn" "PTS526 SK15 SMTR2 LFS"
+			(at 133.35 127 0)
+			(effects
+				(font
+					(size 1.27 1.27)
+				)
+				(hide yes)
+			)
+		)
+		(property "LCSC" "C2689521"
+			(at 133.35 127 0)
+			(effects

Commit message: Doc updated
Other:
- company: (none) -> Daniel Vilas
- title: (none) -> STM32F103 Devel
Changed lines of the file:
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@@
 	(generator_version "8.0")
 	(paper "A4")
+	(title_block
+		(title "STM32F103 Devel")
+		(date "2024-08-19")
+		(rev "0.0.3")
+		(company "Daniel Vilas")
+	)
 	(junction
 		(at 228.6 34.29)

Commit message: Update MPNS and check
Parts:
- U?: Manufacturer STM32F103CBT7 -> STM32F103CBT6; mpn STM32F103CBT7 -> STM32F103CBT6
Changed lines of the file:
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@@
 			)
 		)
-		(property "Manufacturer" "STM32F103CBT7"
+		(property "Manufacturer" "STM32F103CBT6"
 			(at 49.53 81.28 0)
 			(effects
@@
 			)
 		)
-		(property "mpn" "STM32F103CBT7"
+		(property "mpn" "STM32F103CBT6"
 			(at 49.53 81.28 0)
 			(effects

Commit message: 6Pin conector debug
Parts:
- added J7: Conn_01x06, Connector_PinHeader_2.54mm:PinHeader_1x06_P2.54mm_Vertical, symbol Connector_Generic:Conn_01x06
Connections:
- net GND: now also J7.3 (Pin_3)
- net NRST: now also J7.5 (Pin_5)
- net PA13: now also J7.4 (Pin_4)
- net PA14: now also J7.2 (Pin_2)
- net PB3: now also J7.6 (Pin_6)
- net VCC: now also J7.1 (Pin_1)
Other:
- moved on the sheet: J?
