File: STM32F1/STM32F103/STM32F103CBT8_Devel/usb.kicad_sch (KiCad schematic)
At the start: 6 parts, among them J2 USB_B_Micro

Commit message: MPN from 030
Parts:
- D4: LCSC C2480 -> C2480; Manufacturer (none) -> Würth Elektronik
- R10, R8, R9: Manufacturer (none) -> Bourns Inc.
- R7: Manufacturer (none) -> Bourns Inc.; mnp (none) -> CR0805-FX-1003ELF
Changed lines of the file:
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@@
+			)
+		)
+		(property "Manufacturer" ""
+			(at 41.91 50.8 0)
+			(effects
+				(font
+					(size 1.27 1.27)
+				)
+				(hide yes)
+			)
+		)
+		(property "mnp" ""
+			(at 41.91 50.8 0)
+			(effects
+				(font
+					(size 1.27 1.27)
+				)
+				(hide yes)
 			)
 		)
@@
 			)
 		)
+		(property "Manufacturer" "Bourns Inc."
+			(at 53.34 60.96 0)
+			(effects
+				(font
+					(size 1.27 1.27)
+				)
+				(hide yes)
+			)
+		)
+		(property "mnp" "CR0805-FX-1003ELF"
+			(at 53.34 60.96 0)
+			(effects
+				(font
+					(size 1.27 1.27)
+				)
+				(hide yes)
+			)
+		)
 		(pin "1"
 		)
@@
 			)
 		)
+		(property "Manufacturer" "Bourns Inc."
+			(at 76.2 50.8 0)
+			(effects
+				(font
+					(size 1.27 1.27)
+				)
+				(hide yes)
+			)
+		)
+		(property "mnp" ""
+			(at 76.2 50.8 0)
+			(effects
+				(font
+					(size 1.27 1.27)
+				)
+				(hide yes)
+			)
+		)
 		(pin "1"
 		)
@@
 		)
 		(property "LCSC" "C17544"
+			(at 76.2 53.34 0)
+			(effects
+				(font
+					(size 1.27 1.27)
+				)
+				(hide yes)
+			)
+		)
+		(property "Manufacturer" "Bourns Inc."
+			(at 76.2 53.34 0)
+			(effects
+				(font
+					(size 1.27 1.27)
+				)
+				(hide yes)
+			)
+		)
+		(property "mnp" ""
 			(at 76.2 53.34 0)
 			(effects
@@
 			)
 		)
+		(property "Manufacturer" "Bourns Inc."
+			(at 68.58 44.45 0)
+			(effects
+				(font
+					(size 1.27 1.27)
+				)
+				(hide yes)
+			)
+		)
+		(property "mnp" ""
+			(at 68.58 44.45 0)
+			(effects
+				(font
+					(size 1.27 1.27)
+				)
+				(hide yes)
+			)
+		)
 		(pin "1"
 		)
@@
 			)
 		)
-		(property "LCSC" " C2480"
+		(property "LCSC" "C2480"
 			(at 55.88 45.72 0)
 			(effects
+				(font
+					(size 1.27 1.27)
+				)
+				(hide yes)
+			)
+		)
+		(property "Manufacturer" "Würth Elektronik"
+			(at 55.88 45.72 0)
+			(effects
+				(font
+					(size 1.27 1.27)
+				)
+				(hide yes)
+			)
+		)
+		(property "mnp" ""
+			(at 55.88 45.72 0)
+			(effects

Commit message: Mpn ids
Parts:
- D4: Manufacturer Würth Elektronik -> onsemi; mnp (none) -> SS14
- J2: LCSC (none) -> C2894326; Manufacturer (none) -> Würth Elektronik; mnp (none) -> 629105150521
- R10, R9: mnp (none) -> CR0805-FX-20R0ELF
- R8: mnp (none) -> CR0805-FX-1501ELF
Changed lines of the file:
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@@
 			)
 		)
-		(property "Manufacturer" ""
+		(property "Manufacturer" "Würth Elektronik"
 			(at 41.91 50.8 0)
 			(effects
@@
 			)
 		)
-		(property "mnp" ""
+		(property "mnp" "629105150521"
+			(at 41.91 50.8 0)
+			(effects
+				(font
+					(size 1.27 1.27)
+				)
+				(hide yes)
+			)
+		)
+		(property "LCSC" "C2894326"
 			(at 41.91 50.8 0)
 			(effects
@@
 			)
 		)
-		(property "mnp" ""
+		(property "mnp" "CR0805-FX-20R0ELF"
 			(at 76.2 50.8 0)
 			(effects
@@
 			)
 		)
-		(property "mnp" ""
+		(property "mnp" "CR0805-FX-20R0ELF"
 			(at 76.2 53.34 0)
 			(effects
@@
 			)
 		)
-		(property "mnp" ""
+		(property "mnp" "CR0805-FX-1501ELF"
 			(at 68.58 44.45 0)
 			(effects
@@
 			)
 		)
-		(property "Manufacturer" "Würth Elektronik"
+		(property "Manufacturer" "onsemi"
 			(at 55.88 45.72 0)
 			(effects
@@
 			)
 		)
-		(property "mnp" ""
+		(property "mnp" "SS14"
 			(at 55.88 45.72 0)
 			(effects

Commit message: Mov USB
Connections:
- net VCC_USB: now reaches D4.2 (A), J2.1 (VBUS)
Other:
- moved on the sheet: D4, R10, R7, R8, R9

Commit message: MPN
Parts:
- D4: mnp SS14 -> (none); mpn (none) -> SS14
- J2: mnp 629105150521 -> (none); mpn (none) -> 629105150521
- R10, R9: mnp CR0805-FX-20R0ELF -> (none); mpn (none) -> CR0805-FX-20R0ELF
- R7: mnp CR0805-FX-1003ELF -> (none); mpn (none) -> CR0805-FX-1003ELF
- R8: mnp CR0805-FX-1501ELF -> (none); mpn (none) -> CR0805-FX-1501ELF
Changed lines of the file:
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@@
 			)
 		)
-		(property "mnp" "629105150521"
+		(property "LCSC" "C2894326"
 			(at 41.91 50.8 0)
 			(effects
@@
 			)
 		)
-		(property "LCSC" "C2894326"
+		(property "mpn" "629105150521"
 			(at 41.91 50.8 0)
 			(effects
@@
 			)
 		)
-		(property "mnp" "CR0805-FX-1003ELF"
+		(property "mpn" "CR0805-FX-1003ELF"
 			(at 54.61 60.96 0)
 			(effects
@@
 			)
 		)
-		(property "mnp" "CR0805-FX-20R0ELF"
+		(property "mpn" "CR0805-FX-20R0ELF"
 			(at 77.47 50.8 0)
 			(effects
@@
 			)
 		)
-		(property "mnp" "CR0805-FX-20R0ELF"
+		(property "mpn" "CR0805-FX-20R0ELF"
 			(at 77.47 53.34 0)
 			(effects
@@
 			)
 		)
-		(property "mnp" "CR0805-FX-1501ELF"
+		(property "mpn" "CR0805-FX-1501ELF"
 			(at 69.85 44.45 0)
 			(effects
@@
 			)
 		)
-		(property "mnp" "SS14"
+		(property "mpn" "SS14"
 			(at 57.15 45.72 0)
 			(effects

Commit message: Changes
Parts:
- J2: footprint Connector_USB:USB_Micro-B_Wuerth_629105150521_CircularHoles -> Connector_USB:USB_Micro-B_Amphenol_10118193-0001LF_Horizontal; LCSC C2894326 -> C132562; mpn 629105150521 -> 10118193-0001LF
Changed lines of the file:
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@@
 			)
 		)
-		(property "Footprint" "Connector_USB:USB_Micro-B_Wuerth_629105150521_CircularHoles"
+		(property "Footprint" "Connector_USB:USB_Micro-B_Amphenol_10118193-0001LF_Horizontal"
 			(at 45.72 52.07 0)
 			(effects
@@
 			)
 		)
-		(property "LCSC" "C2894326"
+		(property "LCSC" "C132562"
 			(at 41.91 50.8 0)
 			(effects
@@
 			)
 		)
-		(property "mpn" "629105150521"
+		(property "mpn" "10118193-0001LF"
 			(at 41.91 50.8 0)
 			(effects

Commit message: Doc updated
Other:
- company: (none) -> Daniel Vilas
- title: (none) -> STM32F103 Devel
Changed lines of the file:
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@@
 	(generator_version "8.0")
 	(paper "A4")
+	(title_block
+		(title "STM32F103 Devel")
+		(date "2024-08-19")
+		(rev "0.0.3")
+		(company "Daniel Vilas")
+	)
 	(junction
 		(at 40.64 63.5)
