File: STM32G0/STM32G051/STM32G051C8U6_Devel/STM32G051C8_Devel.sch (KiCad schematic (older format))
At the start: 18 parts, among them J2 Conn_01x04, J4 Conn_01x16, J5 Conn_01x16, J7 Conn_01x04, J8 Conn_01x06, U2 AMS1117-3.3

Commit message: First version of 030
Connections:
- net f_GND is gone; now on net GND: J8.6 (Pin_6)
Changed lines of the file:
@@
 L power:GND #PWR0103
 U 1 1 613F4252
-P 4200 2550
-F 0 "#PWR0103" H 4200 2300 50  0001 C CNN
-F 1 "GND" H 4205 2377 50  0000 C CNN
-F 2 "" H 4200 2550 50  0001 C CNN
-F 3 "" H 4200 2550 50  0001 C CNN
-	1    4200 2550
+P 4200 2500
+F 0 "#PWR0103" H 4200 2250 50  0001 C CNN
+F 1 "GND" H 4205 2327 50  0000 C CNN
+F 2 "" H 4200 2500 50  0001 C CNN
+F 3 "" H 4200 2500 50  0001 C CNN
+	1    4200 2500
 	1    0    0    -1
 $EndComp
