File: STM32F0/STM32F030/STM32F030K6T6TR_Devel/STM32F030K6T6TR_Devel.sch (KiCad schematic (older format))
At the start: 18 parts, among them J1 Conn_01x06, J2 Conn_02x03_Odd_Even, J4 Conn_01x16, J5 Conn_01x16, J7 Conn_02x03_Odd_Even, U2 AMS1117-3.3

Commit message: Kibot Split on files
Parts:
- C10, C14: LCSC C7171 -> C7171
- D1: LCSC C84256 -> C84256
- R2: LCSC C17414 -> C17414
- R4, R6: LCSC C17513 -> C17513
- U2: LCSC C6186 -> C6186
Connections:
- no-connect marks 1 -> 3
Changed lines of the file:
@@
 F 2 "Package_TO_SOT_SMD:SOT-223-3_TabPin2" H 9000 5000 50  0001 C CNN
 F 3 "http://www.advanced-monolithic.com/pdf/ds1117.pdf" H 9100 4550 50  0001 C CNN
-F 4 " C6186" H 9000 4800 50  0001 C CNN "LCSC"
+F 4 "C6186" H 9000 4800 50  0001 C CNN "LCSC"
 	1    9000 4800
 	1    0    0    -1
@@
 F 2 "Capacitor_Tantalum_SMD:CP_EIA-3216-18_Kemet-A" H 9838 4850 50  0001 C CNN
 F 3 "~" H 9800 5000 50  0001 C CNN
-F 4 " C7171" H 9800 5000 50  0001 C CNN "LCSC"
+F 4 "C7171" H 9800 5000 50  0001 C CNN "LCSC"
 	1    9800 5000
 	1    0    0    -1
@@
 F 2 "Capacitor_Tantalum_SMD:CP_EIA-3216-18_Kemet-A" H 8438 4850 50  0001 C CNN
 F 3 "~" H 8400 5000 50  0001 C CNN
-F 4 " C7171" H 8400 5000 50  0001 C CNN "LCSC"
+F 4 "C7171" H 8400 5000 50  0001 C CNN "LCSC"
 	1    8400 5000
 	1    0    0    -1
@@
 F 2 "Resistor_SMD:R_0805_2012Metric" H 7270 1459 50  0001 L CNN
 F 3 "~" H 7200 1550 50  0001 C CNN
-F 4 " C17513" H 7200 1550 50  0001 C CNN "LCSC"
+F 4 "C17513" H 7200 1550 50  0001 C CNN "LCSC"
 	1    7200 1550
 	1    0    0    -1
@@
 F 2 "LED_SMD:LED_0805_2012Metric" H 6800 2000 50  0001 C CNN
 F 3 "~" H 6800 2000 50  0001 C CNN
-F 4 " C84256" V 6800 2000 50  0001 C CNN "LCSC"
+F 4 "C84256" V 6800 2000 50  0001 C CNN "LCSC"
 	1    6800 2000
 	0    -1   -1   0
@@
 F 2 "Resistor_SMD:R_0805_2012Metric" H 6870 1459 50  0001 L CNN
 F 3 "~" H 6800 1550 50  0001 C CNN
-F 4 " C17414" H 6800 1550 50  0001 C CNN "LCSC"
+F 4 "C17414" H 6800 1550 50  0001 C CNN "LCSC"
 	1    6800 1550
 	1    0    0    -1
@@
 F 2 "Resistor_SMD:R_0805_2012Metric" H 7620 1459 50  0001 L CNN
 F 3 "~" H 7550 1550 50  0001 C CNN
-F 4 " C17513" H 7550 1550 50  0001 C CNN "LCSC"
+F 4 "C17513" H 7550 1550 50  0001 C CNN "LCSC"
 	1    7550 1550
 	1    0    0    -1
@@
 	6300 4850 6300 4950
 $Comp
-L power:+5V #PWR?
+L power:+5V #PWR0104
 U 1 1 6146F1A1
 P 4100 4550
-F 0 "#PWR?" H 4100 4400 50  0001 C CNN
+F 0 "#PWR0104" H 4100 4400 50  0001 C CNN
 F 1 "+5V" H 4115 4723 50  0000 C CNN
 F 2 "" H 4100 4550 50  0001 C CNN
@@
 	4100 4700 4100 4800
 $Comp
-L power:GND #PWR?
+L power:GND #PWR0105
 U 1 1 61479B5D
 P 5000 5000
-F 0 "#PWR?" H 5000 4750 50  0001 C CNN
+F 0 "#PWR0105" H 5000 4750 50  0001 C CNN
 F 1 "GND" H 5005 4827 50  0000 C CNN
 F 2 "" H 5000 5000 50  0001 C CNN
@@
 Wire Wire Line
 	5000 4900 5000 4800
+NoConn ~ 4800 3750
+NoConn ~ 4800 3350
 Wire Bus Line
 	1250 4100 1250 5700

Commit message: Uart Changes
Connections:
- net PA10: no longer J1.3 (Pin_3)
- net PA2: now also J1.2 (Pin_2)
- net PA3: now also J1.3 (Pin_3)
- net PA9: no longer J1.2 (Pin_2)
Other:
- note added: "BootLoader (boot0 = 1):\nTX = PA9\nRX = PA10\n\nUART1 default pins:\nTX = PA2\nRX = PA3\n\nLiving la vida loca..."
Changed lines of the file:
@@
 Text Label 4800 3350 2    50   ~ 0
 f_DTR
-Text Label 4550 2700 2    50   ~ 0
+Text Label 4300 900  2    50   ~ 0
 f_RXD
-Text Label 4550 2800 2    50   ~ 0
+Text Label 4300 1000 2    50   ~ 0
 f_TXD
-Text Label 4950 2700 0    50   ~ 0
+Text Label 5600 900  0    50   ~ 0
 PA9
-Text Label 4950 2800 0    50   ~ 0
+Text Label 5600 1000 0    50   ~ 0
 PA10
-Text Label 4750 2700 0    50   ~ 0
-TX
-Text Label 4750 2800 0    50   ~ 0
-RX
+Text Label 5300 900  0    50   ~ 0
+bootTX
+Text Label 5300 1000 0    50   ~ 0
+bootRX
 Wire Wire Line
-	4550 2700 4950 2700
+	5200 900  5600 900
 Wire Wire Line
-	4550 2800 4950 2800
+	5200 1000 5600 1000
 Wire Wire Line
 	4950 3350 4800 3350
@@
 NoConn ~ 4800 3750
 NoConn ~ 4800 3350
+Wire Notes Line
+	3900 700  3900 2000
+Wire Notes Line
+	3900 2000 5950 2000
+Wire Notes Line
+	5950 2000 5950 700
+Wire Notes Line
+	5950 700  3900 700
+Text Notes 4050 1900 0    50   ~ 0
+BootLoader (boot0 = 1):\nTX = PA9\nRX = PA10\n\nUART1 default pins:\nTX = PA2\nRX = PA3\n\nLiving la vida loca...
+Text Label 4500 900  0    50   ~ 0
+TX
+Text Label 4500 1000 0    50   ~ 0
+RX
+Wire Wire Line
+	4300 900  4700 900
+Wire Wire Line
+	4300 1000 4700 1000
+Text Label 4700 900  0    50   ~ 0
+PA2
+Text Label 4700 1000 0    50   ~ 0
+PA3
 Wire Bus Line
 	1250 4100 1250 5700
