File: STM32F0/STM32F030/STM32F030K6T6TR_Devel/STM32F030K6.kicad_sch (KiCad schematic)
At the start: 18 parts, among them J3 Conn_01x06, J6 Conn_02x05 Odd_Even, SW1 SW_Push, SW2 SW_DIP_x02, U1 STM32F030K6Tx, Y1 8MHz

Commit message: Add mpn for pcbway
Parts:
- C11, C6, C7: Manufacturer (none) -> KEMET; mpn (none) -> C0805C104J5RAC7800
- C12, C15: Manufacturer (none) -> KEMET; mpn (none) -> C0805C103J5RAC7210
- C13, C9: Manufacturer (none) -> KEMET; mpn (none) -> C0805C105J4REC7800
- C2, C3: Manufacturer (none) -> KEMET; mpn (none) -> C0805C200J5HAC7800
- J6: Manufacturer (none) -> Amphenol ICC (FCI); mpn (none) -> 20021121-00010C4LF
- L1: Manufacturer (none) -> TDK Corporation; mpn (none) -> MLZ2012N100LT000
- R1, R3: Manufacturer (none) -> Bourns Inc.; mpn (none) -> CR0805-FX-1002ELF
- SW2: Manufacturer (none) -> CTS Electrocomponents; mpn (none) -> CT2192LPST-ND
- U1: Manufacturer (none) -> STMicroelectronics; mpn (none) -> STM32F030K6T6TR
- Y1: Manufacturer (none) -> Abracon LLC; mpn (none) -> ABM3-8.000MHZ-B4Y-T

Commit message: Revision LCSC
Parts:
- J6: LCSC (none) -> C5632705
- SW2: LCSC (none) -> C2842684
Changed lines of the file:
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@@
+			)
+		)
+		(property "LCSC" "C5632705"
+			(at 154.94 38.1 0)
+			(effects
+				(font
+					(size 1.27 1.27)
+				)
+				(hide yes)
 			)
 		)
@@
 			(at 140.97 83.82 0)
 			(effects
+				(font
+					(size 1.27 1.27)
+				)
+				(hide yes)
+			)
+		)
+		(property "LCSC" "C2842684"
+			(at 140.97 83.82 0)
+			(effects
